File: KiCad_Files/ME210_Final_Project.sch (KiCad schematic (older format))
At the start: 15 parts

Commit message: Cleaned up KiCad files
Parts:
- added R?: 50k, symbol Device:R_Small
Connections:
- wire segments 22 -> 24
Other:
- note added: "Beacon"
- note added: "IR Reflection Sensor"
- note removed: "IR Reflection Sensor\nNote: still need to test for R_f value."
- moved on the sheet: C?, R?, U?
Changed lines of the file:
@@
 L Sensor_Proximity:QRE1113 U?
 U 1 1 621167FF
-P 3000 5050
-F 0 "U?" H 3000 5367 50  0000 C CNN
-F 1 "QRB1134" H 3000 5276 50  0000 C CNN
-F 2 "OptoDevice:OnSemi_CASE100AQ" H 3000 4850 50  0001 C CNN
-F 3 "http://www.onsemi.com/pub/Collateral/QRE1113-D.PDF" H 3000 5150 50  0001 C CNN
-	1    3000 5050
-	0    -1   -1   0
+P 3800 4400
+F 0 "U?" H 3800 4717 50  0000 C CNN
+F 1 "QRB1134" H 3800 4626 50  0000 C CNN
+F 2 "OptoDevice:OnSemi_CASE100AQ" H 3800 4200 50  0001 C CNN
+F 3 "http://www.onsemi.com/pub/Collateral/QRE1113-D.PDF" H 3800 4500 50  0001 C CNN
+	1    3800 4400
+	1    0    0    -1
 $EndComp
 Text Notes 2950 3500 0    50   ~ 0
@@
 L pspice:OPAMP U?
 U 1 1 6213B6CD
-P 3850 4550
-F 0 "U?" H 3900 4400 50  0000 L CNN
-F 1 "LM324" H 3850 4300 50  0000 L CNN
-F 2 "" H 3850 4550 50  0001 C CNN
-F 3 "~" H 3850 4550 50  0001 C CNN
-	1    3850 4550
+P 1400 4550
+F 0 "U?" H 1450 4400 50  0000 L CNN
+F 1 "LM324" H 1400 4300 50  0000 L CNN
+F 2 "" H 1400 4550 50  0001 C CNN
+F 3 "~" H 1400 4550 50  0001 C CNN
+	1    1400 4550
 	1    0    0    -1
 $EndComp
@@
 L power:GND #PWR?
 U 1 1 6214E91B
-P 3750 4850
-F 0 "#PWR?" H 3750 4600 50  0001 C CNN
-F 1 "GND" H 3755 4677 50  0000 C CNN
-F 2 "" H 3750 4850 50  0001 C CNN
-F 3 "" H 3750 4850 50  0001 C CNN
-	1    3750 4850
+P 1300 4850
+F 0 "#PWR?" H 1300 4600 50  0001 C CNN
+F 1 "GND" H 1305 4677 50  0000 C CNN
+F 2 "" H 1300 4850 50  0001 C CNN
+F 3 "" H 1300 4850 50  0001 C CNN
+	1    1300 4850
 	1    0    0    -1
 $EndComp
@@
 L power:+5V #PWR?
 U 1 1 6214EFD8
-P 3750 4250
-F 0 "#PWR?" H 3750 4100 50  0001 C CNN
-F 1 "+5V" H 3765 4423 50  0000 C CNN
-F 2 "" H 3750 4250 50  0001 C CNN
-F 3 "" H 3750 4250 50  0001 C CNN
-	1    3750 4250
+P 1300 4250
+F 0 "#PWR?" H 1300 4100 50  0001 C CNN
+F 1 "+5V" H 1315 4423 50  0000 C CNN
+F 2 "" H 1300 4250 50  0001 C CNN
+F 3 "" H 1300 4250 50  0001 C CNN
+	1    1300 4250
 	1    0    0    -1
 $EndComp
@@
 L Device:C_Small C?
 U 1 1 6214FCFF
-P 4050 4250
-F 0 "C?" V 3821 4250 50  0000 C CNN
-F 1 "0.1uF" V 3912 4250 50  0000 C CNN
-F 2 "" H 4050 4250 50  0001 C CNN
-F 3 "~" H 4050 4250 50  0001 C CNN
-	1    4050 4250
-	0    1    1    0
-$EndComp
-Wire Wire Line
-	3750 4250 3950 4250
-Connection ~ 3750 4250
+P 1600 4250
+F 0 "C?" V 1371 4250 50  0000 C CNN
+F 1 "0.1uF" V 1462 4250 50  0000 C CNN
+F 2 "" H 1600 4250 50  0001 C CNN
+F 3 "~" H 1600 4250 50  0001 C CNN
+	1    1600 4250
+	0    1    1    0
+$EndComp
+Wire Wire Line
+	1300 4250 1500 4250
+Connection ~ 1300 4250
 $Comp
 L power:GND #PWR?
 U 1 1 621513AD
-P 4150 4250
-F 0 "#PWR?" H 4150 4000 50  0001 C CNN
-F 1 "GND" V 4155 4122 50  0000 R CNN
-F 2 "" H 4150 4250 50  0001 C CNN
-F 3 "" H 4150 4250 50  0001 C CNN
-	1    4150 4250
+P 1700 4250
+F 0 "#PWR?" H 1700 4000 50  0001 C CNN
+F 1 "GND" V 1705 4122 50  0000 R CNN
+F 2 "" H 1700 4250 50  0001 C CNN
+F 3 "" H 1700 4250 50  0001 C CNN
+	1    1700 4250
 	0    -1   -1   0
 $EndComp
@@
 L power:GND #PWR?
 U 1 1 62154FCC
-P 3450 4200
-F 0 "#PWR?" H 3450 3950 50  0001 C CNN
-F 1 "GND" H 3455 4027 50  0000 C CNN
-F 2 "" H 3450 4200 50  0001 C CNN
-F 3 "" H 3450 4200 50  0001 C CNN
-	1    3450 4200
-	-1   0    0    1
-$EndComp
-Wire Wire Line
-	3550 4450 3450 4450
-Wire Wire Line
-	3450 4450 3450 4200
-Wire Wire Line
-	3100 4750 3100 4650
-Wire Wire Line
-	3100 4650 3550 4650
+P 1000 4200
+F 0 "#PWR?" H 1000 3950 50  0001 C CNN
+F 1 "GND" H 1005 4027 50  0000 C CNN
+F 2 "" H 1000 4200 50  0001 C CNN
+F 3 "" H 1000 4200 50  0001 C CNN
+	1    1000 4200
+	-1   0    0    1
+$EndComp
+Wire Wire Line
+	1100 4450 1000 4450
+Wire Wire Line
+	1000 4450 1000 4200
+Wire Wire Line
+	4100 4500 4200 4500
+Wire Wire Line
+	650  4650 1100 4650
 $Comp
 L Device:R_Small R?
 U 1 1 6215949B
-P 3750 5400
-F 0 "R?" V 3946 5400 50  0000 C CNN
-F 1 "R_f" V 3855 5400 50  0000 C CNN
-F 2 "" H 3750 5400 50  0001 C CNN
-F 3 "~" H 3750 5400 50  0001 C CNN
-	1    3750 5400
-	0    -1   -1   0
-$EndComp
-Wire Wire Line
-	3550 4650 3550 5400
-Wire Wire Line
-	3550 5400 3650 5400
-Connection ~ 3550 4650
-Wire Wire Line
-	3850 5400 4150 5400
-Wire Wire Line
-	4150 5400 4150 4550
+P 1300 5400
+F 0 "R?" V 1496 5400 50  0000 C CNN
+F 1 "R_f" V 1405 5400 50  0000 C CNN
+F 2 "" H 1300 5400 50  0001 C CNN
+F 3 "~" H 1300 5400 50  0001 C CNN
+	1    1300 5400
+	0    -1   -1   0
+$EndComp
+Wire Wire Line
+	1100 4650 1100 5400
+Wire Wire Line
+	1100 5400 1200 5400
+Connection ~ 1100 4650
+Wire Wire Line
+	1400 5400 1700 5400
+Wire Wire Line
+	1700 5400 1700 4550
 $Comp
 L power:+5V #PWR?
 U 1 1 6215A70B
-P 2900 4650
-F 0 "#PWR?" H 2900 4500 50  0001 C CNN
-F 1 "+5V" H 2915 4823 50  0000 C CNN
-F 2 "" H 2900 4650 50  0001 C CNN
-F 3 "" H 2900 4650 50  0001 C CNN
-	1    2900 4650
-	1    0    0    -1
-$EndComp
-Wire Wire Line
-	2900 4650 2900 4750
+P 4300 3850
+F 0 "#PWR?" H 4300 3700 50  0001 C CNN
+F 1 "+5V" H 4315 4023 50  0000 C CNN
+F 2 "" H 4300 3850 50  0001 C CNN
+F 3 "" H 4300 3850 50  0001 C CNN
+	1    4300 3850
+	1    0    0    -1
+$EndComp
 Text GLabel 8400 5750 2    50   Output ~ 0
 LineSensor_1
-Text GLabel 4250 4550 2    50   Output ~ 0
+Text GLabel 4350 4300 2    50   Output ~ 0
 LineSensor_1
 Wire Wire Line
-	4150 4550 4250 4550
-Connection ~ 4150 4550
+	1700 4550 1800 4550
+Connection ~ 1700 4550
 $Comp
 L power:+5V #PWR?
 U 1 1 6215F953
-P 2900 5550
-F 0 "#PWR?" H 2900 5400 50  0001 C CNN
-F 1 "+5V" H 2915 5723 50  0000 C CNN
-F 2 "" H 2900 5550 50  0001 C CNN
-F 3 "" H 2900 5550 50  0001 C CNN
-	1    2900 5550
-	-1   0    0    1
+P 3300 4300
+F 0 "#PWR?" H 3300 4150 50  0001 C CNN
+F 1 "+5V" H 3315 4473 50  0000 C CNN
+F 2 "" H 3300 4300 50  0001 C CNN
+F 3 "" H 3300 4300 50  0001 C CNN
+	1    3300 4300
+	0    -1   -1   0
 $EndComp
 $Comp
 L Device:R_Small R?
 U 1 1 621601A5
-P 2900 5450
-F 0 "R?" H 2700 5500 50  0000 L CNN
-F 1 "100" H 2700 5400 50  0000 L CNN
-F 2 "" H 2900 5450 50  0001 C CNN
-F 3 "~" H 2900 5450 50  0001 C CNN
-	1    2900 5450
-	1    0    0    -1
+P 3400 4300
+F 0 "R?" H 3200 4350 50  0000 L CNN
+F 1 "100" H 3200 4250 50  0000 L CNN
+F 2 "" H 3400 4300 50  0001 C CNN
+F 3 "~" H 3400 4300 50  0001 C CNN
+	1    3400 4300
+	0    1    1    0
 $EndComp
 $Comp
 L power:GND #PWR?
 U 1 1 62160D09
-P 3100 5350
-F 0 "#PWR?" H 3100 5100 50  0001 C CNN
-F 1 "GND" H 3105 5177 50  0000 C CNN
-F 2 "" H 3100 5350 50  0001 C CNN
-F 3 "" H 3100 5350 50  0001 C CNN
-	1    3100 5350
-	1    0    0    -1
-$EndComp
-Text Notes 2800 3900 0    50   ~ 0
-IR Reflection Sensor\nNote: still need to test for R_f value.
+P 3500 4500
+F 0 "#PWR?" H 3500 4250 50  0001 C CNN
+F 1 "GND" H 3505 4327 50  0000 C CNN
+F 2 "" H 3500 4500 50  0001 C CNN
+F 3 "" H 3500 4500 50  0001 C CNN
+	1    3500 4500
+	0    1    1    0
+$EndComp
+Text Notes 3350 3900 0    50   ~ 0
+IR Reflection Sensor
 Text Notes 650  850  0    118  ~ 24
 MINIMUM VIABLE PRODUCT SCHEMATIC
+Text Notes 1100 3800 0    50   ~ 0
+Beacon
+$Comp
+L power:GND #PWR?
+U 1 1 62163155
+P 4200 4500
+F 0 "#PWR?" H 4200 4250 50  0001 C CNN
+F 1 "GND" H 4205 4327 50  0000 C CNN
+F 2 "" H 4200 4500 50  0001 C CNN
+F 3 "" H 4200 4500 50  0001 C CNN
+	1    4200 4500
+	0    -1   -1   0
+$EndComp
+$Comp
+L Device:R_Small R?
+U 1 1 62165126
+P 4300 3950
+F 0 "R?" H 4100 4000 50  0000 L CNN
+F 1 "50k" H 4100 3900 50  0000 L CNN
+F 2 "" H 4300 3950 50  0001 C CNN
+F 3 "~" H 4300 3950 50  0001 C CNN
+	1    4300 3950
+	-1   0    0    1
+$EndComp
+Wire Wire Line
+	4350 4300 4300 4300
+Wire Wire Line
+	4300 4050 4300 4300
+Connection ~ 4300 4300
+Wire Wire Line
+	4300 4300 4100 4300
 $EndSCHEMATC

Commit message: added sensor class, editing beacon sensor on kicad
Parts:
- added C?: 200pF, symbol Device:C_Small
- added C?: 147pF, symbol Device:C_Small
- added Q? (x3): LTR-3208E, symbol Device:Q_Photo_NPN
- added R? (x2): 50k, symbol Device:R_Small
- added R? (x2): 1k, symbol Device:R_Small
- added R? (x3): 10k, symbol Device:R_Small
- added U?: LM324, symbol pspice:OPAMP
- gave numbers to parts that had none: 1
Connections:
- wire segments 24 -> 45
Other:
- note added: "Line Sensor 1"
- note added: "Red Becon Sensing\n(3333 Hz)"
- note added: "Red Becon Sensing\n(909 Hz)"
- note removed: "IR Reflection Sensor"
- moved on the sheet: 33k, C?, R?, U?
